Commit message: v1.1

File: rover_description/urdf/arm/gripper.urdf.xacro (robot description, xacro)
@@ -9,4 +9,15 @@
           <mesh filename="package://rover_description/meshes/dae/Cube.013.dae" scale="0.50000 1.00000 2.50000"/>
         </geometry>
+        <surface>
+          <friction>
+            <ode>
+              <mu>1.000000</mu>
+              <mu2>1.000000</mu2>
+              <fdir1>0.000000 0.000000 1.000000</fdir1>
+              <slip1>0.0050000</slip1>
+              <slip2>0.0050000</slip2>
+            </ode>
+          </friction>
+        </surface>
       </collision>
       <inertial>
@@ -29,4 +40,15 @@
           <mesh filename="package://rover_description/meshes/dae/Cube.035.dae" scale="0.50000 1.00000 2.50000"/>
         </geometry>
+        <surface>
+          <friction>
+            <ode>
+              <mu>1.000000</mu>
+              <mu2>1.000000</mu2>
+              <fdir1>0.000000 0.000000 1.000000</fdir1>
+              <slip1>0.0050000</slip1>
+              <slip2>0.0050000</slip2>
+            </ode>
+          </friction>
+        </surface>
       </collision>
       <inertial>
@@ -55,4 +77,5 @@
       <child link="${prefix}_pinza1_link"/>
       <axis xyz="0 0 1"/>
+      <dynamics damping="1.0" friction="1.0"/>
     </joint>
     <joint name="${prefix}_pinza2_link_joint" type="prismatic">
@@ -62,4 +85,5 @@
       <child link="${prefix}_pinza2_link"/>
       <axis xyz="0 0 1"/>
+      <dynamics damping="1.0" friction="1.0"/>
     </joint>
   </xacro:macro>
